File: PCB/HerbUnitPCB/peripherals.kicad_sch (KiCad schematic)
At the start: 15 parts, among them J3 Conn_01x03_Pin, J4 SD_Card_Device, J5 Screw_Terminal_01x02, J6 Conn_01x03_Pin, SW3 SW_Push, U5 DHT11

Commit message: Started PCB design
- Assigned footprints to remaining components
- Brought components into PCB editor and laid them out in general groups
Parts:
- D2, D3, D4: footprint (none) -> LED_SMD:LED_0201_0603Metric
- J4: footprint Connector_Card:SD_Card_Device_16mm_SlotDepth -> Connector_Card:SD_Hirose_DM1AA_SF_PEJ82
Changed lines of the file:
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@@
 			)
 		)
-		(property "Footprint" "Connector_Card:SD_Card_Device_16mm_SlotDepth"
+		(property "Footprint" "Connector_Card:SD_Hirose_DM1AA_SF_PEJ82"
 			(at 149.86 83.82 0)
 			(hide yes)
@@
 			)
 		)
-		(property "Footprint" ""
+		(property "Footprint" "LED_SMD:LED_0201_0603Metric"
 			(at 49.53 46.99 0)
 			(hide yes)
@@
 			)
 		)
-		(property "Footprint" ""
+		(property "Footprint" "LED_SMD:LED_0201_0603Metric"
 			(at 49.53 33.02 0)
 			(hide yes)
@@
 			)
 		)
-		(property "Footprint" ""
+		(property "Footprint" "LED_SMD:LED_0201_0603Metric"
 			(at 49.53 59.69 0)
 			(hide yes)

Commit message: Arranged components
Parts:
- D2, D3, D4: footprint LED_SMD:LED_0201_0603Metric -> LED_SMD:LED_1210_3225Metric_Pad1.42x2.65mm_HandSolder
- J3, J6: footprint (none) -> Connector_PinHeader_2.54mm:PinHeader_1x03_P2.54mm_Horizontal
- J5: footprint (none) -> TerminalBlock_Philmore:TerminalBlock_Philmore_TB132_1x02_P5.00mm_Horizontal
- R14, R9: footprint Resistor_SMD:R_0402_1005Metric -> Resistor_SMD:R_0805_2012Metric
Changed lines of the file:
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@@
 			)
 		)
-		(property "Footprint" ""
+		(property "Footprint" "TerminalBlock_Philmore:TerminalBlock_Philmore_TB132_1x02_P5.00mm_Horizontal"
 			(at 69.85 96.52 0)
 			(hide yes)
@@
 			)
 		)
-		(property "Footprint" "LED_SMD:LED_0201_0603Metric"
+		(property "Footprint" "LED_SMD:LED_1210_3225Metric_Pad1.42x2.65mm_HandSolder"
 			(at 49.53 46.99 0)
 			(hide yes)
@@
 			)
 		)
-		(property "Footprint" "LED_SMD:LED_0201_0603Metric"
+		(property "Footprint" "LED_SMD:LED_1210_3225Metric_Pad1.42x2.65mm_HandSolder"
 			(at 49.53 33.02 0)
 			(hide yes)
@@
 			)
 		)
-		(property "Footprint" "Resistor_SMD:R_0402_1005Metric"
+		(property "Footprint" "Resistor_SMD:R_0805_2012Metric"
 			(at 61.214 98.044 90)
 			(hide yes)
@@
 			)
 		)
-		(property "Footprint" ""
+		(property "Footprint" "Connector_PinHeader_2.54mm:PinHeader_1x03_P2.54mm_Horizontal"
 			(at 48.26 127 0)
 			(hide yes)
@@
 			)
 		)
-		(property "Footprint" "Resistor_SMD:R_0402_1005Metric"
+		(property "Footprint" "Resistor_SMD:R_0805_2012Metric"
 			(at 147.574 31.496 90)
 			(hide yes)
@@
 			)
 		)
-		(property "Footprint" "LED_SMD:LED_0201_0603Metric"
+		(property "Footprint" "LED_SMD:LED_1210_3225Metric_Pad1.42x2.65mm_HandSolder"
 			(at 49.53 59.69 0)
 			(hide yes)
@@
 			)
 		)
-		(property "Footprint" ""
+		(property "Footprint" "Connector_PinHeader_2.54mm:PinHeader_1x03_P2.54mm_Horizontal"
 			(at 153.67 40.64 0)
 			(hide yes)
