File: PCB/HerbUnitPCB/peripherals.kicad_sch (KiCad schematic)
At the start: 15 parts, among them J3 Conn_01x03_Pin, J4 SD_Card_Device, J5 Screw_Terminal_01x02, J6 Conn_01x03_Pin, SW3 CalibrationButton, U5 DHT11

Commit message: Fixed component errors.
Parts:
- J4: MPN MSD-3-A -> DM1AA-SF-PEJ(21); Manufacturer Same Sky -> Hirose Electric Co Ltd
Changed lines of the file:
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@@
 			)
 		)
-		(property "MPN" "  MSD-3-A"
+		(property "MPN" "DM1AA-SF-PEJ(21)"
 			(at 149.86 83.82 0)
 			(hide yes)
@@
 			)
 		)
-		(property "Manufacturer" "Same Sky"
+		(property "Manufacturer" "Hirose Electric Co Ltd"
 			(at 149.86 83.82 0)
 			(hide yes)
