File: PCB/HerbUnitPCB/ESP32_S3.kicad_sch (KiCad schematic)
At the start: 30 parts, among them J1 USB_C_Receptacle_USB2.0_16P, J2 Barrel_Jack_Switch_Pin3Ring, SW1 SW_Push, SW2 SW_Push, U1 USBLC6-2P6, U2 ESP32-S3-WROOM-1, U3 AMS1117-5.0, U6 AP2112K-3.3

Commit message: Changed LED footprints
Thnx Robert :)
Parts:
- D5, D6: value Green LED -> Green
Changed lines of the file:
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@@
 			)
 		)
-		(property "Value" "Green LED"
-			(at 109.982 144.272 90)
+		(property "Value" "Green"
+			(at 114.808 144.272 90)
 			(show_name no)
 			(do_not_autoplace no)
@@
 			)
 		)
-		(property "Value" "Green LED"
+		(property "Value" "Green"
 			(at 182.372 143.51 90)
 			(show_name no)
